File: PCB files/blossom_pcb/arisu.kicad_pcb (KiCad board)
At the start: 2 copper layers, 339.1 x 118.7 mm, 191 parts, among them J1 USB_B_Micro, J10 PF6, J11 PF7, J12 VCC, J13 D+, J14 D-, J15 GND, J2 MISO, J3 VCC, J4 SCK, J5 MOSI, J6 RES, J7 GND, J8 PF4, J9 PF5, SW1 SW_Push, SW10 SW_Push, SW11 SW_Push, SW12 SW_Push, SW13 SW_Push, SW14 SW_Push, SW15 SW_Push, SW16 SW_Push, SW17 SW_Push, SW18 SW_Push, SW19 SW_Push, SW2 SW_Push, SW20 SW_Push, SW21 SW_Push, SW22 SW_Push, SW23 SW_Push, SW24 SW_Push, SW25 SW_Push, SW26 SW_Push, SW27 SW_Push, SW28 SW_Push, SW29 SW_Push, SW3 SW_Push, SW30 SW_Push, SW31 SW_Push, SW32 SW_Push, SW33 SW_Push, SW34 SW_Push, SW35 SW_Push, SW36 SW_Push, SW37 SW_Push, SW38 SW_Push, SW39 SW_Push, SW4 SW_Push, SW40 SW_Push, SW41 SW_Push, SW42 SW_Push, SW43 SW_Push, SW44 SW_Push, SW45 SW_Push, SW46 SW_Push, SW47 SW_Push, SW48 SW_Push, SW49 SW_Push, SW5 SW_Push, SW50 SW_Push, SW51 SW_Push, SW52 SW_Push, SW53 SW_Push, SW54 SW_Push, SW55 SW_Push, SW56 SW_Push, SW57 SW_Push, SW58 SW_Push, SW59 SW_Push, SW6 SW_Push, SW60 SW_Push, SW61 SW_Push, SW62 SW_Push, SW63 SW_Push, SW64 SW_Push, SW65 SW_Push, SW66 SW_Push, SW67 SW_Push, SW7 SW_Push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

Commit message: added rp2040, need to update footprints
Connections:
- net /~RES~ renamed /~{RES}
Other:
- net class Default removed
- net class Power removed

Commit message: Almost doing stuffs
Parts:
- removed J10: PF6, Pin_Headers:Pin_Header_Straight_1x01_Pitch2.54mm
- removed J11: PF7, Pin_Headers:Pin_Header_Straight_1x01_Pitch2.54mm
- removed J12, J3: VCC, Pin_Headers:Pin_Header_Straight_1x01_Pitch2.54mm
- removed J13: D+, Pin_Headers:Pin_Header_Straight_1x01_Pitch2.54mm
- removed J14: D-, Pin_Headers:Pin_Header_Straight_1x01_Pitch2.54mm
- removed J15, J7: GND, Pin_Headers:Pin_Header_Straight_1x01_Pitch2.54mm
- removed J2: MISO, Pin_Headers:Pin_Header_Straight_1x01_Pitch2.54mm
- removed J4: SCK, Pin_Headers:Pin_Header_Straight_1x01_Pitch2.54mm
- removed J5: MOSI, Pin_Headers:Pin_Header_Straight_1x01_Pitch2.54mm
- removed J6: RES, Pin_Headers:Pin_Header_Straight_1x01_Pitch2.54mm
- removed J8: PF4, Pin_Headers:Pin_Header_Straight_1x01_Pitch2.54mm
- removed J9: PF5, Pin_Headers:Pin_Header_Straight_1x01_Pitch2.54mm
- removed SWR1: SW_Push, Buttons_Switches_SMD:SW_SPST_TL3342
- added C10: 100n, Capacitor_SMD:C_0402_1005Metric, B.Cu at (-159.5, 63.5)
- added C11: 100n, Capacitor_SMD:C_0402_1005Metric, B.Cu at (-149.4, 68.6)
- added C12: 1u, Capacitor_SMD:C_0402_1005Metric, B.Cu at (-159.5, 68.6)
- added C13: 100n, Capacitor_SMD:C_0402_1005Metric, B.Cu at (-167.2, 77.0)
- added C14: 100n, Capacitor_SMD:C_0402_1005Metric, B.Cu at (-167.2, 79.0)
- added C15: 100n, Capacitor_SMD:C_0402_1005Metric, B.Cu at (-167.2, 81.0)
- added C16: 100n, Capacitor_SMD:C_0402_1005Metric, B.Cu at (-167.2, 82.9)
- added C17: 10u, Capacitor_SMD:C_0805_2012Metric, B.Cu at (-199.1, 89.8)
- added D101: WS2812B, LED_SMD:LED_WS2812B_PLCC4_5.0x5.0mm_P3.2mm, B.Cu at (-155.0, -77.1)
- added D102: WS2812B, LED_SMD:LED_WS2812B_PLCC4_5.0x5.0mm_P3.2mm, B.Cu at (-155.0, -70.5)
- added D103: WS2812B, LED_SMD:LED_WS2812B_PLCC4_5.0x5.0mm_P3.2mm, B.Cu at (-155.0, -63.9)
- added D104: WS2812B, LED_SMD:LED_WS2812B_PLCC4_5.0x5.0mm_P3.2mm, B.Cu at (-155.0, -57.2)
- added D105: WS2812B, LED_SMD:LED_WS2812B_PLCC4_5.0x5.0mm_P3.2mm, B.Cu at (-146.6, -77.1)
- added D106: WS2812B, LED_SMD:LED_WS2812B_PLCC4_5.0x5.0mm_P3.2mm, B.Cu at (-146.6, -70.5)
- added D107: WS2812B, LED_SMD:LED_WS2812B_PLCC4_5.0x5.0mm_P3.2mm, B.Cu at (-146.6, -63.9)
- added D108: WS2812B, LED_SMD:LED_WS2812B_PLCC4_5.0x5.0mm_P3.2mm, B.Cu at (-146.6, -57.2)
- added D109: WS2812B, LED_SMD:LED_WS2812B_PLCC4_5.0x5.0mm_P3.2mm, B.Cu at (-138.2, -77.1)
- added D110: WS2812B, LED_SMD:LED_WS2812B_PLCC4_5.0x5.0mm_P3.2mm, B.Cu at (-138.2, -70.5)
- added D111: WS2812B, LED_SMD:LED_WS2812B_PLCC4_5.0x5.0mm_P3.2mm, B.Cu at (-138.2, -63.9)
- added D112: WS2812B, LED_SMD:LED_WS2812B_PLCC4_5.0x5.0mm_P3.2mm, B.Cu at (-138.2, -57.2)
- added D113: WS2812B, LED_SMD:LED_WS2812B_PLCC4_5.0x5.0mm_P3.2mm, B.Cu at (-129.8, -77.1)
- added D114: WS2812B, LED_SMD:LED_WS2812B_PLCC4_5.0x5.0mm_P3.2mm, B.Cu at (-129.8, -70.5)
- added D115: WS2812B, LED_SMD:LED_WS2812B_PLCC4_5.0x5.0mm_P3.2mm, B.Cu at (-129.8, -63.9)
- added D116: WS2812B, LED_SMD:LED_WS2812B_PLCC4_5.0x5.0mm_P3.2mm, B.Cu at (-129.8, -57.2)
- added D84: WS2812B, LED_SMD:LED_WS2812B_PLCC4_5.0x5.0mm_P3.2mm, B.Cu at (-180.2, 47.3)
- added H10: MountingHole, MountingHole:MountingHole_2.2mm_M2_Pad, F.Cu at (-225.0, 33.0)
- added H11: MountingHole, MountingHole:MountingHole_2.2mm_M2_Pad, F.Cu at (-219.1, 27.1)
- added H12: MountingHole, MountingHole:MountingHole_2.2mm_M2_Pad, F.Cu at (-219.1, 33.0)
- added H9: MountingHole, MountingHole:MountingHole_2.2mm_M2_Pad, F.Cu at (-225.0, 27.1)
- added R101: 500, Resistor_SMD:R_0805_2012Metric, B.Cu at (-160.0, 15.2)
- added R6: 27, Capacitor_SMD:C_0402_1005Metric, B.Cu at (-159.5, 81.3)
- added R7: 500, Resistor_SMD:R_0805_2012Metric, B.Cu at (-207.4, 52.0)
- added REF**: Stabilizer_Cherry_MX_2.00u, PCM_Mounting_Keyboard_Stabilizer:Stabilizer_Cherry_MX_2.00u, F.Cu at (89.5, -136.9)
- added REF**: Stabilizer_Cherry_MX_2.00u, PCM_Mounting_Keyboard_Stabilizer:Stabilizer_Cherry_MX_2.00u, F.Cu at (215.9, -136.9)
- added REF**: Stabilizer_Cherry_MX_2.00u, PCM_Mounting_Keyboard_Stabilizer:Stabilizer_Cherry_MX_2.00u, F.Cu at (106.0, -127.3)
- added REF**: Stabilizer_Cherry_MX_2.00u, PCM_Mounting_Keyboard_Stabilizer:Stabilizer_Cherry_MX_2.00u, F.Cu at (199.4, -127.3)
- added SW68: SW_Push, PCM_Switch_Keyboard_Hotswap_Kailh:SW_Hotswap_Kailh_MX_1.00u, F.Cu at (194.8, 121.5)
- added SW69: SW_Push, PCM_Switch_Keyboard_Hotswap_Kailh:SW_Hotswap_Kailh_MX_1.00u, F.Cu at (226.6, 121.5)
- added SW70: SW_Push, PCM_Switch_Keyboard_Hotswap_Kailh:SW_Hotswap_Kailh_MX_1.00u, F.Cu at (236.2, 138.0)
- added SW71: SW_Push, PCM_Switch_Keyboard_Hotswap_Kailh:SW_Hotswap_Kailh_MX_1.00u, F.Cu at (245.7, 154.5)
- added SW72: SW_Push, PCM_Switch_Keyboard_Hotswap_Kailh:SW_Hotswap_Kailh_MX_1.00u, F.Cu at (301.2, 113.1)
- added SW73: SW_Push, PCM_Switch_Keyboard_Hotswap_Kailh:SW_Hotswap_Kailh_MX_1.00u, F.Cu at (320.3, 110.7)
- added SW74: SW_Push, PCM_Switch_Keyboard_Hotswap_Kailh:SW_Hotswap_Kailh_MX_1.00u, F.Cu at (339.3, 113.1)
- added SW75: SW_Push, PCM_Switch_Keyboard_Hotswap_Kailh:SW_Hotswap_Kailh_MX_1.00u, F.Cu at (358.4, 117.9)
- added SW76: SW_Push, PCM_Switch_Keyboard_Hotswap_Kailh:SW_Hotswap_Kailh_MX_1.00u, F.Cu at (377.4, 117.9)
- added U3: RP2040, RP2040_minimal:RP2040-QFN-56, B.Cu at (-186.3, 73.9)
- C1, C2: value 22pF -> 27p; footprint Capacitors_SMD:C_0805_HandSoldering -> Capacitor_SMD:C_0402_1005Metric
- C3: value 10uF -> 10u; footprint Capacitors_SMD:C_0805_HandSoldering -> Capacitor_SMD:C_0805_2012Metric
- C4: value 1uF (±10%) -> 100n; footprint Capacitors_SMD:C_0805_HandSoldering -> Capacitor_SMD:C_0402_1005Metric
- C5: value 1uF -> 10u; footprint Capacitors_SMD:C_0805_HandSoldering -> Capacitor_SMD:C_0805_2012Metric
- C6, C7, C9: value 0.1uF -> 100n; footprint Capacitors_SMD:C_0805_HandSoldering -> Capacitor_SMD:C_0402_1005Metric
- C8: value 0.1uF -> 1u; footprint Capacitors_SMD:C_0805_HandSoldering -> Capacitor_SMD:C_0402_1005Metric
- D1, D10, D11, D12, D13, D14, D15, D16, D17, D18, D19, D2, D20, D21, D22, D23, D24, D25, D26, D27, D28, D29, D3, D30, D31, D32, D33, D34, D35, D36, D37, D38, D39, D4, D40, D41, D42, D43, D44, D45, D46, D47, D48, D49, D5, D50, D51, D52, D53, D54, D55, D56, D57, D58, D59, D6, D60, D61, D62, D63, D64, D65, D66, D67, D7, D8, D9: footprint Diodes_SMD:D_SOD-123 -> Diode_SMD:D_SOD-123
- D68, D69, D70, D71, D72, D73, D75, D76: value WS2812B -> D; footprint LED_SMD:LED_WS2812B_PLCC4_5.0x5.0mm_P3.2mm -> Diode_SMD:D_SOD-123
- D74: value WS2812B -> D; footprint LED_SMD:LED_WS2812B_PLCC4_5.0x5.0mm_P3.2mm -> Diode_SMD:D_SOD-123; moved to B.Cu
- D78: moved to B.Cu
- H1, H2, H3, H4: footprint Mounting_Holes:MountingHole_2.2mm_M2_Pad -> MountingHole:MountingHole_2.7mm_M2.5
- H5, H6, H7, H8: footprint Mounting_Holes:MountingHole_2.2mm_M2_Pad -> MountingHole:MountingHole_2.2mm_M2_Pad
- J1: value USB_B_Micro -> Conn_01x02; footprint Connectors_USB:USB_Micro-B_Molex-105017-0001 -> Connector_PinHeader_2.54mm:PinHeader_1x02_P2.54mm_Vertical
- R1: value 22 -> 1k; footprint Resistors_SMD:R_0805_HandSoldering -> Capacitor_SMD:C_0402_1005Metric
- R2: value 22 -> DNF; footprint Resistors_SMD:R_0805_HandSoldering -> Capacitor_SMD:C_0402_1005Metric
- R3: value 10K -> 1k; footprint Resistors_SMD:R_0805_HandSoldering -> Capacitor_SMD:C_0402_1005Metric
- R4: footprint Resistors_SMD:R_0805_HandSoldering -> Resistor_SMD:R_0805_2012Metric
- R5: value 500 -> 27; footprint Resistor_SMD:R_0805_2012Metric -> Capacitor_SMD:C_0402_1005Metric
- SW1, SW10, SW11, SW12, SW13, SW15, SW16, SW17, SW18, SW19, SW20, SW21, SW22, SW24, SW25, SW26, SW27, SW28, SW29, SW30, SW31, SW32, SW33, SW34, SW35, SW36, SW38, SW39, SW40, SW41, SW42, SW43, SW44, SW45, SW47, SW48, SW49, SW50, SW51, SW52, SW53, SW55, SW56, SW58, SW59, SW6, SW61, SW62, SW63, SW64, SW65, SW66, SW67, SW7, SW8, SW9: footprint MX_Switch:SW_Cherry_MX_1.00u_PCB -> PCM_Switch_Keyboard_Hotswap_Kailh:SW_Hotswap_Kailh_MX_1.00u
- SW14, SW2, SW46, SW5, SW60: footprint MX_Switch:SW_Cherry_MX_1.50u_PCB -> PCM_Switch_Keyboard_Hotswap_Kailh:SW_Hotswap_Kailh_MX_1.00u
- SW23: footprint MX_Switch:SW_Cherry_MX_2.00u_PCB_ReversedStabilizers -> PCM_Switch_Keyboard_Hotswap_Kailh:SW_Hotswap_Kailh_MX_1.00u
- SW3, SW54: footprint MX_Switch:SW_Cherry_MX_1.75u_PCB -> PCM_Switch_Keyboard_Hotswap_Kailh:SW_Hotswap_Kailh_MX_1.00u
- SW37: footprint MX_Switch:SW_Cherry_MX_2.75u_PCB_ReversedStabilizers -> PCM_Switch_Keyboard_Hotswap_Kailh:SW_Hotswap_Kailh_MX_1.00u
- SW4: footprint MX_Switch:SW_Cherry_MX_2.25u_PCB -> PCM_Switch_Keyboard_Hotswap_Kailh:SW_Hotswap_Kailh_MX_1.00u
- SW57: footprint MX_Switch:SW_Cherry_MX_2.25u_PCB_ReversedStabilizers -> PCM_Switch_Keyboard_Hotswap_Kailh:SW_Hotswap_Kailh_MX_1.00u
- U1: value USBLC6-2SC6 -> NCP1117-3.3_SOT223; footprint TO_SOT_Packages_SMD:SOT-23-6_Handsoldering -> Package_TO_SOT_SMD:SOT-223-3_TabPin2
- U2: value ATmega32U4-AU -> W25Q128JVS; footprint Housings_QFP:TQFP-44_10x10mm_Pitch0.8mm -> Package_SO:SOIC-8_5.23x5.23mm_P1.27mm
- Y1: value Crystal_GND24 -> ABLS-12.000MHZ-B4-T; footprint Crystals:Crystal_SMD_SeikoEpson_FA238-4pin_3.2x2.5mm_HandSoldering -> RP2040_minimal:Crystal_SMD_HC49-US
- moved H8 581.5 mm to (-231.0, 33.0)
- moved H7 572.4 mm to (-231.0, 27.1)
- moved D82 536.8 mm to (-180.2, 34.0), turned to 180 degrees
- moved D78 488.1 mm to (-188.6, 34.0), turned to 180 degrees
- moved H6 485.9 mm to (-236.9, 33.0)
- moved H5 466.1 mm to (-236.9, 27.1)
- moved D79 464.1 mm to (-188.6, 40.6), turned to 180 degrees
- moved D81 422.0 mm to (-180.2, 27.4), turned to 180 degrees
- moved J1 420.9 mm to (-244.5, 54.2), turned to 180 degrees
- moved D83 396.7 mm to (-180.2, 40.6), turned to 180 degrees
- moved U1 391.8 mm to (-223.5, 66.0), turned to 180 degrees
- moved Y1 387.1 mm to (-193.0, 63.5), turned to 180 degrees
- moved D77 380.3 mm to (-188.6, 27.4), turned to 180 degrees
- moved R4 378.3 mm to (-208.3, 68.6), turned to 180 degrees
- moved H3 365.4 mm to (-243.4, 41.5)
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Connections:
- C1 pad 1: GND -> Net-(Y1-Pin_2)
- C1 pad 2: XTAL1 -> GND
- C2 pad 1: XTAL2 -> Net-(C2-Pad1)
- C3 pad 1: VCC -> VBUS
- C4 pad 1: Net-(C4-Pad1) -> +3V3
- C5 pad 1: VCC -> +3V3
- C6 pad 1: VCC -> +1V1
- C7 pad 1: VCC -> +1V1
- C8 pad 1: VCC -> +1V1
- C9 pad 1: VCC -> +3V3
- D1 pad 1: /row0 -> /GPIO5
- D10 pad 1: /row0 -> Net-(D10-K)
- D11 pad 1: /row1 -> Net-(D10-K)
- D12 pad 1: /row2 -> Net-(D10-K)
- D13 pad 1: /row3 -> Net-(D10-K)
- D14 pad 1: /row4 -> Net-(D10-K)
- D15 pad 1: /row0 -> /GPIO6
- D16 pad 1: /row1 -> /GPIO6
- D17 pad 1: /row2 -> /GPIO6
- D18 pad 1: /row3 -> /GPIO6
- D19 pad 1: /row0 -> /GPIO6
- D2 pad 1: /row1 -> /GPIO5
- D20 pad 1: /row1 -> /GPIO6
- D21 pad 1: /row2 -> /GPIO6
- D22 pad 1: /row3 -> Net-(D22-K)
- D23 pad 1: /row4 -> Net-(D22-K)
- D24 pad 1: /row0 -> Net-(D22-K)
- D25 pad 1: /row1 -> Net-(D22-K)
- D26 pad 1: /row2 -> Net-(D22-K)
- D27 pad 1: /row3 -> Net-(D22-K)
- D28 pad 1: /row4 -> Net-(D22-K)
- D29 pad 1: /row0 -> /GPIO7
- D3 pad 1: /row2 -> /GPIO5
- D30 pad 1: /row1 -> /GPIO7
- D31 pad 1: /row2 -> /GPIO7
- D32 pad 1: /row3 -> /GPIO7
- D33 pad 1: /row0 -> /GPIO7
- D34 pad 1: /row1 -> /GPIO7
- D35 pad 1: /row2 -> /GPIO7
- D36 pad 1: /row3 -> /GPIO7
- D37 pad 1: /row4 -> /GPIO7
- D38 pad 1: /row0 -> /GPIO7
- D39 pad 1: /row1 -> /GPIO7
- D4 pad 1: /row3 -> /GPIO5
- D40 pad 1: /row2 -> /GPIO7
- D41 pad 1: /row3 -> /GPIO7
- D42 pad 1: /row0 -> /GPIO7
- D43 pad 1: /row1 -> /GPIO7
- D44 pad 1: /row2 -> /GPIO7
- D45 pad 1: /row3 -> /GPIO8
- D46 pad 1: /row4 -> /GPIO8
- D47 pad 1: /row0 -> /GPIO8
- D48 pad 1: /row1 -> /GPIO8
- D49 pad 1: /row2 -> /GPIO8
- D5 pad 1: /row4 -> /GPIO5
- D50 pad 1: /row3 -> /GPIO8
- D51 pad 1: /row0 -> /GPIO8
- D52 pad 1: /row1 -> /GPIO8
- D53 pad 1: /row2 -> /GPIO8
- D54 pad 1: /row3 -> /GPIO8
- D55 pad 1: /row0 -> /GPIO8
- D56 pad 1: /row1 -> /GPIO8
- D57 pad 1: /row2 -> /GPIO8
- D58 pad 1: /row4 -> /GPIO8
- D59 pad 1: /row0 -> /GPIO8
- D6 pad 1: /row0 -> /GPIO5
- D60 pad 1: /row1 -> /GPIO8
- D61 pad 1: /row3 -> /GPIO9
- D62 pad 1: /row4 -> /GPIO9
- D63 pad 1: /row0 -> /GPIO9
- D64 pad 1: /row1 -> /GPIO9
- D65 pad 1: /row2 -> /GPIO9
- D66 pad 1: /row3 -> /GPIO9
- D67 pad 1: /row4 -> /GPIO9
- D68 pad 1: VCC -> /GPIO9
- D68 pad 2: Net-(D68-Pad2) -> Net-(D68-A)
- D69 pad 1: VCC -> /GPIO9
- D69 pad 2: Net-(D69-Pad2) -> Net-(D69-A)
- D7 pad 1: /row1 -> /GPIO5
- D70 pad 1: VCC -> /GPIO9
- D70 pad 2: Net-(D70-Pad2) -> Net-(D70-A)
- D71 pad 1: VCC -> /GPIO9
- D71 pad 2: Net-(D71-Pad2) -> Net-(D71-A)
- D72 pad 1: VCC -> /GPIO9
- D72 pad 2: Net-(D72-Pad2) -> Net-(D72-A)
- D73 pad 1: VCC -> /GPIO9
- D73 pad 2: Net-(D73-Pad2) -> Net-(D73-A)
- D74 pad 1: VCC -> /GPIO9
- D74 pad 2: Net-(D74-Pad2) -> Net-(D74-A)
- D75 pad 1: VCC -> /GPIO9
- D75 pad 2: Net-(D75-Pad2) -> Net-(D75-A)
- D76 pad 1: VCC -> /GPIO9
- D76 pad 2: Net-(D76-Pad2) -> Net-(D76-A)
- D77 pad 4: Net-(D73-Pad2) -> Net-(D73-DOUT)
- D78 pad 4: Net-(D74-Pad2) -> Net-(D74-DOUT)
- D79 pad 4: Net-(D75-Pad2) -> Net-(D75-DOUT)
- D8 pad 1: /row2 -> Net-(D10-K)
- D80 pad 2: Net-(D69-Pad4) -> Net-(D80-DOUT)
- D80 pad 4: Net-(D76-Pad2) -> Net-(D76-DOUT)
- D81 pad 2: Net-(D70-Pad4) -> Net-(D70-DIN)
- D82 pad 2: Net-(D71-Pad4) -> Net-(D71-DIN)
- D9 pad 1: /row3 -> Net-(D10-K)
- J1 pad 1: VCC -> /~{USB_BOOT}
- J1 pad 2: Net-(J1-Pad2) -> GND
- R1 pad 1: D+ -> /QSPI_SS
- R1 pad 2: Net-(J1-Pad3) -> /~{USB_BOOT}
- R2 pad 1: D- -> +3V3
- R2 pad 2: Net-(J1-Pad2) -> /QSPI_SS
- R3 pad 1: VCC -> /XOUT
- R3 pad 2: /~{RES} -> Net-(C2-Pad1)
- R4 pad 1: Net-(R4-Pad1) -> +3V3
- R4 pad 2: GND -> /RUN
- R5 pad 1: /PF4 -> /USB_D+
- R5 pad 2: Net-(D68-Pad4) -> Net-(U3-USB_DP)
- SW1 pad 1: /col0 -> /GPIO10
- SW10 pad 1: /col2 -> /GPIO21
- SW11 pad 1: /col2 -> /GPIO22
- SW12 pad 1: /col2 -> /GPIO23
- SW13 pad 1: /col2 -> /GPIO24
- SW14 pad 1: /col2 -> /GPIO25
- SW15 pad 1: /col3 -> /GPIO10
- SW16 pad 1: /col3 -> /GPIO11
- SW17 pad 1: /col3 -> /GPIO12
- SW18 pad 1: /col3 -> /GPIO13
- SW19 pad 1: /col4 -> /GPIO14
- SW2 pad 1: /col0 -> /GPIO11
- SW20 pad 1: /col4 -> /GPIO15
- SW21 pad 1: /col4 -> /GPIO16
- SW22 pad 1: /col4 -> /GPIO19
- SW23 pad 1: /col4 -> /GPIO20
- SW24 pad 1: /col5 -> /GPIO21
- SW25 pad 1: /col5 -> /GPIO22
- SW26 pad 1: /col5 -> /GPIO23
- SW27 pad 1: /col5 -> /GPIO24
- SW28 pad 1: /col5 -> /GPIO25
- SW29 pad 1: /col6 -> /GPIO10
- SW3 pad 1: /col0 -> /GPIO12
- SW30 pad 1: /col6 -> /GPIO11
- SW31 pad 1: /col6 -> /GPIO12
- SW32 pad 1: /col6 -> /GPIO13
- SW33 pad 1: /SCK -> /GPIO14
- SW34 pad 1: /SCK -> /GPIO15
- SW35 pad 1: /SCK -> /GPIO16
- SW36 pad 1: /SCK -> /GPIO17
- SW37 pad 1: /SCK -> /GPIO18
- SW38 pad 1: /col8 -> /GPIO19
- SW39 pad 1: /col8 -> /GPIO20
- SW4 pad 1: /col0 -> /GPIO13
- SW40 pad 1: /col8 -> /GPIO21
- SW41 pad 1: /col8 -> /GPIO22
- SW42 pad 1: /col9 -> /GPIO23
- SW43 pad 1: /col9 -> /GPIO24
- SW44 pad 1: /col9 -> /GPIO25
- SW45 pad 1: /col9 -> /GPIO10
- SW46 pad 1: /col9 -> /GPIO11
- SW47 pad 1: /col10 -> /GPIO12
- SW48 pad 1: /col10 -> /GPIO13
- SW49 pad 1: /col10 -> /GPIO14
- SW5 pad 1: /col0 -> /GPIO14
- SW50 pad 1: /col10 -> /GPIO15
- SW51 pad 1: /col11 -> /GPIO16
- SW52 pad 1: /col11 -> /GPIO17
- SW53 pad 1: /col11 -> /GPIO18
- SW54 pad 1: /col11 -> /GPIO19
- SW55 pad 1: /col12 -> /GPIO20
- SW56 pad 1: /col12 -> /GPIO21
- SW57 pad 1: /col12 -> /GPIO22
- SW58 pad 1: /col12 -> /GPIO23
- SW59 pad 1: /col13 -> /GPIO24
- SW6 pad 1: /col1 -> /GPIO15
- SW60 pad 1: /col13 -> /GPIO25
- SW61 pad 1: /col13 -> /GPIO10
- SW62 pad 1: /col13 -> /GPIO11
- SW63 pad 1: /MISO -> /GPIO12
- SW64 pad 1: /MISO -> /GPIO13
- SW65 pad 1: /MISO -> /GPIO14
- SW66 pad 1: /MISO -> /GPIO15
- SW67 pad 1: /MISO -> /GPIO16
- SW7 pad 1: /col1 -> /GPIO16
- SW8 pad 1: /col1 -> /GPIO19
- SW9 pad 1: /col1 -> /GPIO20
- U1 pad 1: Net-(U1-Pad1) -> GND
- U1 pad 2: GND -> +3V3
- U1 pad 3: Net-(U1-Pad3) -> VBUS
- U2 pad 1: /col2 -> /QSPI_SS
- U2 pad 2: VCC -> /QSPI_SD1
- U2 pad 3: D- -> /QSPI_SD2
- U2 pad 4: D+ -> GND
- U2 pad 5: GND -> /QSPI_SD0
- U2 pad 6: Net-(C4-Pad1) -> /QSPI_SCLK
- U2 pad 7: VCC -> /QSPI_SD3
- U2 pad 8: /col8 -> +3V3
- Y1 pad 1: XTAL1 -> /XIN
- Y1 pad 2: GND -> Net-(Y1-Pin_2)
Routing:
- net VCC: track 940.7 -> 0.00 mm, vias 28 -> 0
- net GND: track 807.8 -> 0.00 mm, vias 25 -> 0
- net /row4: track 433.8 -> 0.00 mm, vias 2 -> 0
- net /row3: track 433.6 -> 0.00 mm, vias 2 -> 0
- net /row2: track 399.4 -> 0.00 mm, vias 4 -> 0
- net /row1: track 384.1 -> 0.00 mm, vias 4 -> 0
- net /row0: track 328.0 -> 0.00 mm, vias 4 -> 0
- net /MISO: track 273.4 -> 0.00 mm, vias 1 -> 0
- net /col13: track 269.0 -> 0.00 mm
- net /col12: track 249.0 -> 0.00 mm
- net /col11: track 230.6 -> 0.00 mm
- net /col10: track 221.3 -> 0.00 mm
- net /col0: track 206.6 -> 0.00 mm
- net /col2: track 179.0 -> 0.00 mm, vias 2 -> 0
- net /col1: track 168.2 -> 0.00 mm, vias 2 -> 0
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- removed copper zone on B.Cu, net GND
- removed copper zone on F.Cu, net GND
Other:
- board outline removed
- board text removed: "DouKB"
- board text removed: "Fate Design Rev 1.1"

Commit message: diodes placed
Parts:
- moved D58 291.8 mm to (346.9, 84.1)
- moved D63 288.2 mm to (89.7, 103.2)
- moved D64 279.2 mm to (108.7, 100.8)
- moved D48 261.8 mm to (108.7, 81.8)
- moved D47 257.6 mm to (89.7, 84.1)
- moved D54 254.7 mm to (258.9, 123.8), turned to -150 degrees
- moved D57 254.4 mm to (327.8, 81.8)
- moved D55 237.7 mm to (289.7, 86.5)
- moved D53 212.4 mm to (244.6, 99.1), turned to -150 degrees
- moved D50 202.2 mm to (146.8, 86.5)
- moved D76 188.9 mm to (385.0, 107.9), turned to 180 degrees
- moved D49 186.7 mm to (127.8, 84.1)
- moved D71 175.8 mm to (247.2, 141.6), turned to -150 degrees
- moved D66 174.9 mm to (187.8, 149.5), turned to 150 degrees
- moved D75 171.8 mm to (365.9, 107.9), turned to 180 degrees
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
Commit message: Almost complete
Parts:
- removed D109, D110, D111, D112, D113, D114, D115, D116, D77, D78, D79, D80, D81, D82, D83, D84: WS2812B, LED_SMD:LED_WS2812B_PLCC4_5.0x5.0mm_P3.2mm
- removed R7: 500, Resistor_SMD:R_0805_2012Metric
- R4: moved to F.Cu
- moved D102 529.6 mm to (365.9, 24.6)
- moved D103 500.2 mm to (308.0, 125.4)
- moved J1 466.4 mm to (221.5, 33.6)
- moved D104 435.9 mm to (217.5, 169.1)
- moved U1 420.2 mm to (196.1, 43.7)
- moved D105 402.2 mm to (171.4, 169.1)
- moved D101 400.7 mm to (232.6, 24.6)
- moved R4 394.0 mm to (185.7, 65.1), turned to 0 degrees
- moved C10 389.7 mm to (230.2, 62.7)
- moved C17 389.7 mm to (189.1, 54.8)
- moved U2 389.5 mm to (219.1, 48.4), turned to 90 degrees
- moved C12 385.0 mm to (225.4, 65.9)
- moved U3 382.1 mm to (195.6, 61.0)
- moved C3 381.8 mm to (203.2, 46.0), turned to 0 degrees
- moved R1 380.7 mm to (225.4, 41.3), turned to 90 degrees
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- renumbered REF** to SW36_Stab1, REF** to SW37_Stab1, REF** to SW51_Stab1, REF** to SW54_Stab1
Connections:
- D10 pad 1: Net-(D10-K) -> /GPIO5
- D108 pad 2: Net-(D108-DOUT) -> unconnected-(D108-DOUT-Pad2)
- D11 pad 1: Net-(D10-K) -> /GPIO5
- D12 pad 1: Net-(D10-K) -> /GPIO5
- D13 pad 1: Net-(D10-K) -> /GPIO5
- D14 pad 1: Net-(D10-K) -> /GPIO5
- D22 pad 1: Net-(D22-K) -> /GPIO6
- D23 pad 1: Net-(D22-K) -> /GPIO6
- D24 pad 1: Net-(D22-K) -> /GPIO6
- D25 pad 1: Net-(D22-K) -> /GPIO6
- D26 pad 1: Net-(D22-K) -> /GPIO6
- D27 pad 1: Net-(D22-K) -> /GPIO6
- D28 pad 1: Net-(D22-K) -> /GPIO6
- D8 pad 1: Net-(D10-K) -> /GPIO5
- D9 pad 1: Net-(D10-K) -> /GPIO5
Routing:
- net VCC: track 0.00 -> 674.1 mm
- net /GPIO8: track 0.00 -> 523.0 mm, vias 0 -> 4
- net /GPIO9: track 0.00 -> 502.0 mm, vias 0 -> 2
- net /GPIO7: track 0.00 -> 475.5 mm, vias 0 -> 6
- net /GPIO5: track 0.00 -> 372.3 mm, vias 0 -> 4
- net /GPIO6: track 0.00 -> 369.6 mm, vias 0 -> 3
- net /GPIO10: track 0.00 -> 313.8 mm, vias 0 -> 8
- net /GPIO25: track 0.00 -> 299.4 mm, vias 0 -> 6
- net /GPIO11: track 0.00 -> 279.6 mm, vias 0 -> 6
- net /GPIO24: track 0.00 -> 275.5 mm, vias 0 -> 6
- net /GPIO12: track 0.00 -> 261.4 mm, vias 0 -> 13
- net /GPIO23: track 0.00 -> 253.0 mm, vias 0 -> 6
- net /GPIO15: track 0.00 -> 233.9 mm, vias 0 -> 8
- net /GPIO22: track 0.00 -> 232.1 mm, vias 0 -> 6
- net /GPIO19: track 0.00 -> 230.0 mm, vias 0 -> 6
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- added copper zone on F.Cu, net GND
Other:
- board outline added: 369.9 x 155.6 mm

Commit message: Everything is connected
Parts:
- moved R6 26.6 mm to (201.6, 50.8), turned to -90 degrees
- moved R5 8.29 mm to (203.2, 50.8), turned to -90 degrees
Routing:
- net /GPIO20: track 176.9 -> 256.2 mm
- net /GPIO7: track 475.5 -> 545.5 mm, vias 6 -> 8
- net /GPIO17: track 127.3 -> 62.3 mm, vias 6 -> 2
- net +1V1: track 7.96 -> 49.7 mm, vias 0 -> 4
- net +3V3: track 138.8 -> 169.4 mm, vias 2 -> 3
- net Net-(U3-USB_DM): track 0.00 -> 11.5 mm
- net Net-(U3-USB_DP): track 4.43 -> 12.6 mm
- net Net-(D61-A): track 5.79 -> 0.00 mm
- net Net-(D65-A): track 5.00 -> 0.00 mm
- net Net-(D63-A): track 5.00 -> 0.00 mm
- net Net-(D62-A): track 5.00 -> 0.00 mm
- net Net-(D5-A): track 5.00 -> 0.00 mm
- net Net-(D49-A): track 5.00 -> 0.00 mm
- net Net-(D47-A): track 5.00 -> 0.00 mm
- net Net-(D46-A): track 5.00 -> 0.00 mm
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
Commit message: Adjusted rp2040 layout and changed pin assignments
Parts:
- moved C10 33.0 mm to (211.1, 89.7)
- moved C11 31.2 mm to (211.1, 97.6)
- moved C12 31.2 mm to (211.1, 93.7)
- moved C17 18.6 mm to (179.4, 38.9)
- moved R2 18.4 mm to (228.9, 51.6), turned to 90 degrees
- moved C9 14.8 mm to (211.1, 100.8)
- moved J1 14.1 mm to (229.4, 45.2), turned to 90 degrees
- moved C5 12.4 mm to (179.4, 42.1)
- moved R1 8.67 mm to (228.9, 49.2)
- moved C3 8.39 mm to (195.3, 43.2)
- moved U1 8.39 mm to (188.2, 40.9)
- moved C2 4.76 mm to (187.8, 69.7)
- moved R3 4.69 mm to (190.2, 69.7), turned to 180 degrees
- moved R4 2.03 mm to (187.7, 64.5)
- turned C6 to 0 degrees
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Connections:
- SW17 pad 1: /GPIO12 -> /GPIO18
- SW18 pad 1: /GPIO13 -> /GPIO19
- SW19 pad 1: /GPIO14 -> /GPIO20
- SW20 pad 1: /GPIO15 -> /GPIO17
- SW22 pad 1: /GPIO19 -> /GPIO13
- SW23 pad 1: /GPIO20 -> /GPIO12
- SW3 pad 1: /GPIO12 -> /GPIO18
- SW31 pad 1: /GPIO12 -> /GPIO18
- SW32 pad 1: /GPIO13 -> /GPIO19
- SW33 pad 1: /GPIO14 -> /GPIO20
- SW34 pad 1: /GPIO15 -> /GPIO17
- SW36 pad 1: /GPIO17 -> /GPIO15
- SW37 pad 1: /GPIO18 -> /GPIO14
- SW38 pad 1: /GPIO19 -> /GPIO13
- SW39 pad 1: /GPIO20 -> /GPIO12
- SW4 pad 1: /GPIO13 -> /GPIO19
- SW47 pad 1: /GPIO12 -> /GPIO18
- SW48 pad 1: /GPIO13 -> /GPIO19
- SW49 pad 1: /GPIO14 -> /GPIO20
- SW5 pad 1: /GPIO14 -> /GPIO20
- SW50 pad 1: /GPIO15 -> /GPIO17
- SW52 pad 1: /GPIO17 -> /GPIO15
- SW53 pad 1: /GPIO18 -> /GPIO14
- SW54 pad 1: /GPIO19 -> /GPIO13
- SW55 pad 1: /GPIO20 -> /GPIO12
- SW6 pad 1: /GPIO15 -> /GPIO17
- SW63 pad 1: /GPIO12 -> /GPIO18
- SW64 pad 1: /GPIO13 -> /GPIO19
- SW65 pad 1: /GPIO14 -> /GPIO20
- SW66 pad 1: /GPIO15 -> /GPIO17
- SW68 pad 1: /GPIO17 -> /GPIO15
- SW69 pad 1: /GPIO18 -> /GPIO14
- SW70 pad 1: /GPIO19 -> /GPIO13
- SW71 pad 1: /GPIO20 -> /GPIO12
- SW8 pad 1: /GPIO19 -> /GPIO13
- SW9 pad 1: /GPIO20 -> /GPIO12
Routing:
- net /GPIO15: track 233.9 -> 57.5 mm, vias 8 -> 3
- net /GPIO20: track 256.2 -> 103.1 mm
- net /GPIO14: track 204.2 -> 66.6 mm, vias 5 -> 3
- net /GPIO19: track 232.5 -> 95.8 mm
- net /GPIO13: track 226.2 -> 89.6 mm, vias 11 -> 6
- net /GPIO12: track 261.4 -> 157.5 mm, vias 13 -> 5
- net /GPIO8: track 522.2 -> 424.0 mm, vias 4 -> 2
- net /GPIO21: track 216.3 -> 125.7 mm, vias 6 -> 2
- net /GPIO24: track 275.7 -> 187.5 mm
- net /GPIO23: track 253.2 -> 165.7 mm
- net /GPIO22: track 232.3 -> 145.7 mm
- net /GPIO25: track 299.5 -> 214.3 mm
- net +3V3: track 169.4 -> 84.8 mm, vias 3 -> 2
- net /GPIO17: track 62.3 -> 146.0 mm, vias 2 -> 6
- net /GPIO7: track 545.5 -> 463.9 mm, vias 8 -> 4
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- added copper zone on B.Cu, net +1V1
- added copper zone on B.Cu, net +3V3
- added copper zone on F.Cu, net /GPIO12
- added copper zone on F.Cu, net /GPIO13
- added copper zone on F.Cu, net /GPIO21
- added copper zone on F.Cu, net /GPIO22
- added copper zone on F.Cu, net /GPIO23
- added copper zone on F.Cu, net /GPIO24
- added copper zone on F.Cu, net /GPIO25
