File: PCB files/blossom_pcb/arisu.kicad_pcb (KiCad board)
At the start: 2 copper layers, 370.5 x 156 mm, 211 parts, among them J1 USB_C_Receptacle_USB2.0, P1 Conn_ARM_JTAG_SWD_10, SW1 SW_Push, SW10 SW_Push, SW11 SW_Push, SW12 SW_Push, SW13 SW_Push, SW14 SW_Push, SW15 SW_Push, SW16 SW_Push, SW17 SW_Push, SW18 SW_Push, SW19 SW_Push, SW2 SW_Push, SW20 SW_Push, SW21 SW_Push, SW22 SW_Push, SW23 SW_Push, SW24 SW_Push, SW25 SW_Push, SW26 SW_Push, SW27 SW_Push, SW28 SW_Push, SW29 SW_Push, SW3 SW_Push, SW30 SW_Push, SW31 SW_Push, SW32 SW_Push, SW33 SW_Push, SW34 SW_Push, SW35 SW_Push, SW36 SW_Push, SW37 SW_Push, SW38 SW_Push, SW39 SW_Push, SW4 SW_Push, SW40 SW_Push, SW41 SW_Push, SW42 SW_Push, SW43 SW_Push, SW44 SW_Push, SW45 SW_Push, SW46 SW_Push, SW47 SW_Push, SW48 SW_Push, SW49 SW_Push, SW5 SW_Push, SW50 SW_Push, SW51 SW_Push, SW52 SW_Push, SW53 SW_Push, SW54 SW_Push, SW55 SW_Push, SW56 SW_Push, SW57 SW_Push, SW58 SW_Push, SW59 SW_Push, SW6 SW_Push, SW60 SW_Push, SW61 SW_Push, SW62 SW_Push, SW63 SW_Push, SW64 SW_Push, SW65 SW_Push, SW66 SW_Push, SW67 SW_Push, SW68 SW_Push, SW69 SW_Push, SW7 SW_Push, SW70 SW_Push, SW71 SW_Push, SW72 SW_Push, SW73 SW_Push, SW74 SW_Push, SW75 SW_Push, SW76 SW_Push, SW8 SW_Push, SW9 SW_Push, U1 XC6206PxxxMR, U2 W25Q128JVS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

Commit message: Final Prototype 1
Connections:
- net SWCLK renamed /SWCLK
- net SWDIO renamed /SWDIO
- P1 pad 1: +5V -> +3V3
- P1 pad 5: GND -> unconnected-(P1-GND-Pad5)
Routing:
- net +5V: track 856.3 -> 819.8 mm, vias 4 -> 3
- net +3V3: track 53.1 -> 65.3 mm, vias 0 -> 1
- net GND: track 93.3 -> 90.2 mm

Commit message: New model and "final" pcb
Parts:
- moved H5 29.6 mm to (402.9, 36.9)
- moved H3 29.5 mm to (401.9, 142.9)
- moved H2 28.1 mm to (218.5, 186.0)
- moved D13 27.9 mm to (369.5, 59.4)
- moved D14 27.9 mm to (393.3, 59.4)
- moved D27 27.9 mm to (369.5, 78.4)
- moved D28 27.9 mm to (393.3, 78.4)
- moved D59 27.9 mm to (369.5, 116.5)
- moved D60 27.9 mm to (393.3, 116.5)
- moved D75 27.9 mm to (369.5, 135.6)
- moved LED2 27.9 mm to (389.9, 38.9)
- moved SW12 27.9 mm to (347.2, 51.2)
- moved SW26 27.9 mm to (347.2, 70.3)
- moved SW58 27.9 mm to (347.2, 108.4)
- moved SW74 27.9 mm to (347.2, 127.4)
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Routing:
- net /col10: track 253.3 -> 263.2 mm
- net /col15: track 276.5 -> 285.6 mm
- net /col14: track 247.5 -> 256.3 mm
- net /col13: track 225.6 -> 233.4 mm
- net /col11: track 187.1 -> 194.3 mm
- net /col12: track 205.3 -> 212.4 mm
- net /col9: track 235.8 -> 242.8 mm
- net GND: track 90.2 -> 93.7 mm, vias 21 -> 20
- net /row3: track 501.9 -> 504.9 mm
- net +5V: track 819.8 -> 817.1 mm
- net Net-(J1-CC1): track 4.16 -> 1.72 mm, vias 1 -> 0
- net Net-(J1-CC2): track 4.56 -> 2.43 mm, vias 1 -> 0
- net /col8: track 174.3 -> 175.7 mm
Other:
- board size 370.5 x 156 mm -> 375 x 157 mm

Commit message: iter1
Parts:
- SW1, SW10, SW11, SW12, SW13, SW14, SW15, SW16, SW17, SW18, SW19, SW2, SW20, SW21, SW22, SW23, SW24, SW25, SW26, SW27, SW28, SW29, SW3, SW30, SW31, SW32, SW33, SW34, SW35, SW36, SW37, SW38, SW39, SW4, SW40, SW41, SW42, SW43, SW44, SW45, SW46, SW47, SW48, SW49, SW5, SW50, SW51, SW52, SW53, SW54, SW55, SW56, SW57, SW58, SW59, SW6, SW60, SW61, SW62, SW63, SW64, SW65, SW66, SW67, SW68, SW69, SW7, SW70, SW71, SW72, SW73, SW74, SW75, SW76, SW8, SW9: moved to B.Cu
- turned SW1 to 180 degrees
- turned SW10 to 180 degrees
- turned SW11 to 180 degrees
- turned SW12 to 180 degrees
- turned SW13 to 180 degrees
- turned SW14 to 180 degrees
- turned SW15 to 180 degrees
- turned SW16 to 180 degrees
- turned SW17 to 180 degrees
- turned SW18 to 180 degrees
- turned SW19 to 180 degrees
- turned SW2 to 180 degrees
- turned SW20 to 180 degrees
- turned SW21 to 180 degrees
- turned SW22 to 180 degrees
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
Commit message: Fixed PCB for LEDs and R9
Parts:
- C1: footprint Capacitor_SMD:C_0402_1005Metric -> Capacitor_SMD:C_0603_1608Metric
- R101: footprint Resistor_SMD:R_0402_1005Metric -> Resistor_SMD:R_1210_3225Metric
- R9: footprint Resistor_SMD:R_0402_1005Metric -> Resistor_SMD:R_0805_2012Metric
- moved R1 6.93 mm to (243.4, 78.7), turned to 0 degrees
- moved R101 2.05 mm to (250.0, 37.3)
- moved R8 2.01 mm to (244.5, 66.0)
- moved C4 2.00 mm to (242.9, 57.0)
- moved R10 2.00 mm to (244.5, 63.9)
- moved U2 2.00 mm to (241.0, 62.7)
- moved R4 1.61 mm to (211.0, 78.1)
- moved R11 1.44 mm to (213.1, 78.1)
- moved R9 0.48 mm to (211.1, 39.6)
- moved C1 0.46 mm to (221.6, 84.0)
- moved C10 0.11 mm to (213.3, 76.1)
- moved C2 0.11 mm to (216.5, 82.2)
- moved C18 0.09 mm to (211.5, 41.2)
Routing:
- net /col7: track 84.9 -> 107.3 mm
- net Net-(LED4-DOUT): track 60.6 -> 52.3 mm
- net Net-(LED6-DOUT): track 186.0 -> 178.1 mm
- net +5V: track 817.1 -> 810.5 mm
- net /QSPI_SS: track 32.2 -> 37.5 mm, vias 2 -> 0
- net /PWM: track 52.9 -> 57.2 mm
- net Net-(BOOT1-Pad2): track 12.3 -> 8.88 mm
- net GND: track 93.7 -> 96.4 mm
- net /row0: track 409.0 -> 411.7 mm
- net /col12: track 212.4 -> 214.8 mm
- net /col9: track 242.8 -> 240.7 mm
- net /QSPI_SD2: track 23.6 -> 21.6 mm
- net /QSPI_SD1: track 24.4 -> 22.4 mm
- net /col8: track 175.7 -> 173.8 mm
- net Net-(LED5-DOUT): track 112.9 -> 111.3 mm
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