File: PCB files/blossom_pcb/arisu.kicad_sch (KiCad schematic)
At the start: 73 parts, among them J1 USB_B_Micro, J10 PF6, J11 PF7, J12 VCC, J13 D+, J14 D-, J15 GND, J2 Conn_01x02, J2 MISO, J3 VCC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

Commit message: added rp2040, need to update footprints
Parts:
- removed C1, C2: 22pF, Capacitor_SMD:C_0805_2012Metric, symbol Device:C
- removed C3: 10uF, Capacitor_SMD:C_0805_2012Metric, symbol Device:C
- removed C4: 1uF (±10%), Capacitor_SMD:C_0805_2012Metric, symbol Device:C
- removed C5: 1uF, Capacitor_SMD:C_0805_2012Metric, symbol Device:C
- removed C6, C7, C8, C9: 0.1uF, Capacitor_SMD:C_0805_2012Metric, symbol Device:C
- removed J1: USB_B_Micro, Connectors_USB:USB_Micro-B_Molex-105017-0001, symbol Connector:USB_B_Micro
- removed J1: USB_B_Micro, RP2040_minimal:USB_Micro-B_Amphenol_10103594-0001LF_Horizontal_modified, symbol RP2040_minimal-rescue:USB_B_Micro-Connector
- removed J10: PF6, Pin_Headers:Pin_Header_Straight_1x01_Pitch2.54mm, symbol Connector_Generic:Conn_01x01
- removed J11: PF7, Pin_Headers:Pin_Header_Straight_1x01_Pitch2.54mm, symbol Connector_Generic:Conn_01x01
- removed J12: VCC, Pin_Headers:Pin_Header_Straight_1x01_Pitch2.54mm, symbol Connector_Generic:Conn_01x01
- removed J13: D+, Pin_Headers:Pin_Header_Straight_1x01_Pitch2.54mm, symbol Connector_Generic:Conn_01x01
- removed J14: D-, Pin_Headers:Pin_Header_Straight_1x01_Pitch2.54mm, symbol Connector_Generic:Conn_01x01
- removed J15: GND, Pin_Headers:Pin_Header_Straight_1x01_Pitch2.54mm, symbol Connector_Generic:Conn_01x01
- removed J2: MISO, Pin_Headers:Pin_Header_Straight_1x01_Pitch2.54mm, symbol Connector_Generic:Conn_01x01
- removed J8: PF4, Pin_Headers:Pin_Header_Straight_1x01_Pitch2.54mm, symbol Connector_Generic:Conn_01x01
- removed J9: PF5, Pin_Headers:Pin_Header_Straight_1x01_Pitch2.54mm, symbol Connector_Generic:Conn_01x01
- removed R1, R2: 22, Resistor_SMD:R_0805_2012Metric, symbol Device:R
- removed R3, R4: 10K, Resistor_SMD:R_0805_2012Metric, symbol Device:R
- removed U1: USBLC6-2SC6, TO_SOT_Packages_SMD:SOT-23-6_Handsoldering, symbol Power_Protection:USBLC6-2SC6
- removed U2: ATmega32U4-AU, Housings_QFP:TQFP-44_10x10mm_Pitch0.8mm, symbol arisu-rescue:ATmega32U4-AU-MCU_Microchip_ATmega
- removed Y1: Crystal_GND24, Crystal:Crystal_SMD_3225-4Pin_3.2x2.5mm, symbol Device:Crystal_GND24
- C?: renamed from C2; symbol Device:C -> arisu-rescue:C-Device
- C?: renamed from C3; symbol Device:C -> arisu-rescue:C-Device
- C?: renamed from C5; symbol Device:C -> arisu-rescue:C-Device
- C?: renamed from C9; symbol Device:C -> arisu-rescue:C-Device
- C?: renamed from C11; symbol Device:C -> arisu-rescue:C-Device
- C?: renamed from C12; symbol Device:C -> arisu-rescue:C-Device
- C?: renamed from C13; symbol Device:C -> arisu-rescue:C-Device
- C?: renamed from C14; symbol Device:C -> arisu-rescue:C-Device
- C?: renamed from C15; symbol Device:C -> arisu-rescue:C-Device
- C?: renamed from C16; symbol Device:C -> arisu-rescue:C-Device
- C?: renamed from C6; symbol Device:C -> arisu-rescue:C-Device
- C?: renamed from C7; symbol Device:C -> arisu-rescue:C-Device
- C?: renamed from C8; symbol Device:C -> arisu-rescue:C-Device
- C?: renamed from C10; symbol Device:C -> arisu-rescue:C-Device
- C?: renamed from C1; symbol Device:C -> arisu-rescue:C-Device
- C?: renamed from C4; symbol Device:C -> arisu-rescue:C-Device
- C?: renamed from C17; symbol Device:C -> arisu-rescue:C-Device
- H10: renamed from H6; symbol Mechanical:MountingHole -> arisu-rescue:MountingHole-Mechanical
- H11: renamed from H7; symbol Mechanical:MountingHole -> arisu-rescue:MountingHole-Mechanical
- H12: renamed from H8; symbol Mechanical:MountingHole -> arisu-rescue:MountingHole-Mechanical
- H5, H?: renamed from H1; symbol Mechanical:MountingHole -> arisu-rescue:MountingHole-Mechanical
- H6, H?: renamed from H2; symbol Mechanical:MountingHole -> arisu-rescue:MountingHole-Mechanical
- H7, H?: renamed from H3; symbol Mechanical:MountingHole -> arisu-rescue:MountingHole-Mechanical
- H8, H?: renamed from H4; symbol Mechanical:MountingHole -> arisu-rescue:MountingHole-Mechanical
- H9: renamed from H5; symbol Mechanical:MountingHole -> arisu-rescue:MountingHole-Mechanical
- J2: renamed from J3; symbol Connector_Generic:Conn_01x01 -> arisu-rescue:Conn_01x01-Connector_Generic
- J3: renamed from J4; symbol Connector_Generic:Conn_01x01 -> arisu-rescue:Conn_01x01-Connector_Generic
- J4: renamed from J5; symbol Connector_Generic:Conn_01x01 -> arisu-rescue:Conn_01x01-Connector_Generic
- J5: renamed from J6; symbol Connector_Generic:Conn_01x01 -> arisu-rescue:Conn_01x01-Connector_Generic
- J6: renamed from J7; symbol Connector_Generic:Conn_01x01 -> arisu-rescue:Conn_01x01-Connector_Generic
- J?: renamed from J2; symbol Connector_Generic:Conn_01x02 -> PCM_RP2040_minimal-rescue:Conn_01x02-Connector_Generic
- R4: renamed from R6; symbol Device:R -> arisu-rescue:R-Device
- R?: renamed from R2; symbol Device:R -> arisu-rescue:R-Device
- R?: renamed from R1; symbol Device:R -> arisu-rescue:R-Device
- R?: renamed from R3; symbol Device:R -> arisu-rescue:R-Device
- R?: renamed from R4; symbol Device:R -> arisu-rescue:R-Device
- R?: renamed from R5; symbol Device:R -> arisu-rescue:R-Device
- SWR1: symbol Switch:SW_Push -> arisu-rescue:SW_Push-Switch
- U?: renamed from U3; symbol MCU_RaspberryPi_RP2040:RP2040 -> PCM_RP2040_minimal-rescue:RP2040
- U?: renamed from U2; symbol RP2040_minimal-rescue:W25Q128JVS-Memory_Flash -> PCM_RP2040_minimal-rescue:W25Q128JVS-Memory_Flash
- U?: renamed from U1; symbol Regulator_Linear:NCP1117-3.3_SOT223 -> PCM_RP2040_minimal-rescue:NCP1117-3.3_SOT223-Regulator_Linear
- Y?: renamed from Y1; symbol Device:Crystal -> PCM_RP2040_minimal-rescue:Conn_01x02-Connector_Generic
Connections:
- net SCK is gone; now on net SWCLK: J3.1 (Pin_1)
- net SWD is gone; now on net SWDIO: U?.25 (SWD)
- net ~{RES} is gone; now on net RUN: J5.1 (Pin_1)
- net RUN: now also SWR1.2
- net at C?.1, R?.2: no longer Y?.2
- net MOSI renamed SWDIO
- no-connect marks 5 -> 0
Other:
- sheet LED_matrix ports: added PWM; removed AVR
- moved on the sheet: J2, J3, J4, J5, J6, SWR1

Commit message: Almost doing stuffs
Parts:
- H10, H11, H12, H5, H6, H7, H8, H9: footprint Mounting_Holes:MountingHole_2.2mm_M2_Pad -> MountingHole:MountingHole_2.2mm_M2_Pad
- U?: symbol PCM_RP2040_minimal-rescue:RP2040 -> MCU_RaspberryPi_RP2040:RP2040
Connections:
- net XIN: no longer C?.1
- net at Y?.2 (Pin_2): now also C?.1
Other:
- sheet matrix ports: added col15; removed none

Commit message: Almost complete
Other:
- moved on the sheet: H?

Commit message: Adjusted rp2040 layout and changed pin assignments
Changed lines of the file:
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@@
     (effects (font (size 1.27 1.27)) (justify left bottom))
   )
-  (label "col9" (at 210.82 127 180) (fields_autoplaced)
+  (label "col3" (at 210.82 127 180) (fields_autoplaced)
     (effects (font (size 1.27 1.27)) (justify right bottom))
   )
@@
     (effects (font (size 1.27 1.27)) (justify right bottom))
   )
-  (label "col8" (at 210.82 124.46 180) (fields_autoplaced)
+  (label "col2" (at 210.82 124.46 180) (fields_autoplaced)
     (effects (font (size 1.27 1.27)) (justify right bottom))
   )
@@
     (effects (font (size 1.27 1.27)) (justify right bottom))
   )
-  (label "col10" (at 210.82 129.54 180) (fields_autoplaced)
+  (label "col4" (at 210.82 129.54 180) (fields_autoplaced)
     (effects (font (size 1.27 1.27)) (justify right bottom))
   )
@@
     (effects (font (size 1.27 1.27)) (justify right bottom))
   )
-  (label "col2" (at 210.82 109.22 180) (fields_autoplaced)
+  (label "col10" (at 210.82 109.22 180) (fields_autoplaced)
     (effects (font (size 1.27 1.27)) (justify right bottom))
   )
@@
     (effects (font (size 1.27 1.27)) (justify right bottom))
   )
-  (label "col7" (at 210.82 121.92 180) (fields_autoplaced)
+  (label "col5" (at 210.82 121.92 180) (fields_autoplaced)
     (effects (font (size 1.27 1.27)) (justify right bottom))
   )
@@
     (effects (font (size 1.27 1.27)) (justify right bottom))
   )
-  (label "col3" (at 210.82 111.76 180) (fields_autoplaced)
-    (effects (font (size 1.27 1.27)) (justify right bottom))
-  )
-  (label "col5" (at 210.82 116.84 180) (fields_autoplaced)
+  (label "col9" (at 210.82 111.76 180) (fields_autoplaced)
+    (effects (font (size 1.27 1.27)) (justify right bottom))
+  )
+  (label "col7" (at 210.82 116.84 180) (fields_autoplaced)
     (effects (font (size 1.27 1.27)) (justify right bottom))
   )
@@
     (effects (font (size 1.27 1.27)) (justify left bottom))
   )
-  (label "col4" (at 210.82 114.3 180) (fields_autoplaced)
-    (effects (font (size 1.27 1.27)) (justify right bottom))
-  )
+  (label "col8" (at 210.82 114.3 180) (fields_autoplaced)
+    (effects (font (size 1.27 1.27)) (justify right bottom))
+  )

Commit message: probably final without usb
Parts:
- removed H5, H6: MountingHole, MountingHole:MountingHole_2.2mm_M2_Pad, symbol arisu-rescue:MountingHole-Mechanical
- removed H? (x4): MountingHole, MountingHole:MountingHole_2.7mm_M2.5, symbol arisu-rescue:MountingHole-Mechanical
- renumbered H7 to H1, H8 to H2, H9 to H3, H10 to H4, H11 to H5, H12 to H6
Connections:
- net GPIO0 renamed col15
- net GPIO1 renamed col14
- net GPIO11 renamed row4
- net GPIO12 renamed row3
- net GPIO13 renamed row2
- net GPIO14 renamed row1
- net GPIO15 renamed row0
- net GPIO16 renamed col8
- net GPIO17 renamed col7
- net GPIO2 renamed col13
- net GPIO23 renamed col6
- net GPIO24 renamed col5
- net GPIO25 renamed col4
- net GPIO26_ADC0 renamed col3
- net GPIO27_ADC1 renamed col2
- net GPIO28_ADC2 renamed col1
- net GPIO29_ADC3 renamed col0
- net GPIO3 renamed col12
- net GPIO4 renamed col11
- net GPIO5 renamed col10
- net GPIO6 renamed col9
- net GPIO7 renamed PWM
Other:
- moved on the sheet: H1, H2, H3, H4, H5, H6

Commit message: Added usb
Parts:
- added H7: MountingHole, MountingHole:MountingHole_2.2mm_M2_Pad, symbol arisu-rescue:MountingHole-Mechanical
- added USB1: USB_C_Plug_USB2.0, symbol Connector:USB_C_Plug_USB2.0
Connections:
- net GND: now also USB1.A1 (GND), USB1.A12 (GND), USB1.B1 (GND), USB1.B12 (GND), USB1.S1 (SHIELD)
- net USB_D+: now also USB1.A6 (D+)
- net USB_D-: now also USB1.A7 (D-)
- net VBUS: now also USB1.A4 (VBUS), USB1.A9 (VBUS), USB1.B4 (VBUS), USB1.B9 (VBUS)
Other:
- moved on the sheet: C?, R?, Y?

Commit message: lots of stuff
Parts:
- removed R?: DNF, Capacitor_SMD:C_0402_1005Metric, symbol arisu-rescue:R-Device
- USB1: footprint (none) -> Connector_USB:USB_C_Receptacle_Molex_105450-0101
Changed lines of the file:
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@@
   (junction (at 121.92 27.94) (diameter 0) (color 0 0 0 0)
   )
-  (junction (at 58.42 179.07) (diameter 0) (color 0 0 0 0)
-  )
   (junction (at 91.44 132.08) (diameter 0) (color 0 0 0 0)
   )
@@
   (junction (at 207.01 39.37) (diameter 0) (color 0 0 0 0)
   )
-  (junction (at 73.66 158.75) (diameter 0) (color 0 0 0 0)
-  )
   (junction (at 45.72 95.25) (diameter 0) (color 0 0 0 0)
   )
@@
     (stroke (width 0) (type default))
   )
-  (wire (pts (xy 58.42 160.02) (xy 58.42 158.75))
-    (stroke (width 0) (type default))
-  )
   (wire (pts (xy 45.72 85.09) (xy 77.47 85.09))
     (stroke (width 0) (type default))
@@
     (stroke (width 0) (type default))
   )
-  (wire (pts (xy 73.66 154.94) (xy 73.66 158.75))
-    (stroke (width 0) (type default))
-  )
-  (wire (pts (xy 73.66 158.75) (xy 73.66 171.45))
+  (wire (pts (xy 73.66 154.94) (xy 73.66 171.45))
     (stroke (width 0) (type default))
   )
@@
     (stroke (width 0) (type default))
   )
-  (wire (pts (xy 58.42 167.64) (xy 58.42 179.07))
-    (stroke (width 0) (type default))
-  )
   (wire (pts (xy 101.6 27.94) (xy 113.03 27.94))
     (stroke (width 0) (type default))
@@
     (stroke (width 0) (type default))
   )
-  (wire (pts (xy 58.42 179.07) (xy 60.96 179.07))
-    (stroke (width 0) (type default))
-  )
   (bus (pts (xy 213.36 86.36) (xy 213.36 88.9))
     (stroke (width 0) (type default))
@@
     (stroke (width 0) (type default))
   )
-  (wire (pts (xy 58.42 158.75) (xy 73.66 158.75))
-    (stroke (width 0) (type default))
-  )
   (wire (pts (xy 207.01 29.21) (xy 207.01 27.94))
     (stroke (width 0) (type default))
@@
     (stroke (width 0) (type default))
   )
-  (wire (pts (xy 46.99 179.07) (xy 58.42 179.07))
+  (wire (pts (xy 46.99 179.07) (xy 60.96 179.07))
     (stroke (width 0) (type default))
   )
@@
     )
   )
-  (symbol (lib_id "arisu-rescue:R-Device") (at 58.42 163.83 0) (unit 1)
-    (in_bom yes) (on_board yes) (dnp no)
-    (property "Reference" "R?" (at 60.198 162.6616 0)
-      (effects (font (size 1.27 1.27)) (justify left))
-    )
-    (property "Value" "DNF" (at 60.198 164.973 0)
-      (effects (font (size 1.27 1.27)) (justify left))
-    )
-    (property "Footprint" "Capacitor_SMD:C_0402_1005Metric" (at 56.642 163.83 90)
-      (effects (font (size 1.27 1.27)) hide)
-    )
-    (property "Datasheet" "~" (at 58.42 163.83 0)
-      (effects (font (size 1.27 1.27)) hide)
-    )
-    (pin "1")
-    (pin "2")
-    (instances
-      (project "RP2040_minimal"
-        (path "/4e80874f-13b9-4886-a592-f501191b7905"
-          (reference "R?") (unit 1)
-        )
-      )
-      (project "arisu"
-        (path "/6a4507f9-fb93-401b-b9e1-9f2bcbbd5186"
-          (reference "R2") (unit 1)
-        )
-      )
-    )
-  )
   (symbol (lib_id "arisu-rescue:R-Device") (at 43.18 179.07 270) (unit 1)
     (in_bom yes) (on_board yes) (dnp no)
@@
     (in_bom yes) (on_board yes) (dnp no) (fields_autoplaced)
     (property "Reference" "USB1" (at 26.67 15.24 0)
-      (effects (font (size 1.27 1.27)))
+      (effects (font (size 1.27 1.27)) hide)
     )
     (property "Value" "USB_C_Plug_USB2.0" (at 26.67 17.78 0)
       (effects (font (size 1.27 1.27)))
     )
-    (property "Footprint" "" (at 30.48 36.83 0)
+    (property "Footprint" "Connector_USB:USB_C_Receptacle_Molex_105450-0101" (at 30.48 36.83 0)
       (effects (font (size 1.27 1.27)) hide)
     )

Commit message: Cleanup
Parts:
- removed J2: VCC, Pin_Headers:Pin_Header_Straight_1x01_Pitch2.54mm, symbol arisu-rescue:Conn_01x01-Connector_Generic
- removed J3: SCK, Pin_Headers:Pin_Header_Straight_1x01_Pitch2.54mm, symbol arisu-rescue:Conn_01x01-Connector_Generic
- removed J4: MOSI, Pin_Headers:Pin_Header_Straight_1x01_Pitch2.54mm, symbol arisu-rescue:Conn_01x01-Connector_Generic
- removed J5: RES, Pin_Headers:Pin_Header_Straight_1x01_Pitch2.54mm, symbol arisu-rescue:Conn_01x01-Connector_Generic
- removed J6: GND, Pin_Headers:Pin_Header_Straight_1x01_Pitch2.54mm, symbol arisu-rescue:Conn_01x01-Connector_Generic
- removed J?: Conn_01x02, Connector_PinHeader_2.54mm:PinHeader_1x02_P2.54mm_Vertical, symbol PCM_RP2040_minimal-rescue:Conn_01x02-Connector_Generic
- added BOOT1: K2-6639DP-B4SW-04, Button_Switch_THT:SW_PUSH_6mm, symbol arisu-rescue:SW_Push-Switch
- added P1: Conn_ARM_JTAG_SWD_10, Connector:JLINK_NEEDLE, symbol Connector:Conn_ARM_JTAG_SWD_10
- added R? (x2): 5.1k, Resistor_SMD:R_01005_0402Metric, symbol arisu-rescue:R-Device
- added R?: 1k, Resistor_SMD:R_01005_0402Metric, symbol arisu-rescue:R-Device
- RST1: renamed from SWR1; value SW_Push -> K2-6639DP-B4SW-04; footprint Buttons_Switches_SMD:SW_SPST_TL3342 -> Button_Switch_THT:SW_PUSH_6mm
- Y?: value ABLS-12.000MHZ-B4-T -> X49SM12MSB2SC; footprint RP2040_minimal:Crystal_SMD_HC49-US -> PCM_Crystal_AKL:Crystal_SMD_HC49-SD
Connections:
- net GND: now also BOOT1.1, P1.3 (GND), P1.5 (GND), P1.9 (GNDDetect), R?.1, R?.1, R?.1; no longer USB1.S1 (SHIELD)
- net RUN: now also P1.10 (~{RESET})
- net SWCLK: now also P1.4 (SWDCLK/TCK)
- net SWDIO: now also P1.2 (SWDIO/TMS)
- net VBUS: now also P1.1 (VTref)
- net at USB1.A5 (CC): now also R?.2
- net at USB1.B5 (VCONN): now also R?.2
- net ~{USB_BOOT}: no longer names the net of R?.2
- net ~{USB_BOOT}: now also BOOT1.2
- new net: R?.2, USB1.S1 (SHIELD)
Other:
- note added: "Make sure R4 and R6 are close to RP2040"
- note removed: "Make sure R3 and R4 are close to RP2040"
