File: PCB files/blossom_pcb/arisu.kicad_sch (KiCad schematic)
At the start: 46 parts, among them J1 USB_C_Receptacle_USB2.0, P1 Conn_ARM_JTAG_SWD_10, U1 XC6206PxxxMR, U4 SRV05-4, Y1 Crystal_GND24

Commit message: Possible final
Parts:
- F1: LCSC (none) -> C20803
- J1: LCSC (none) -> C165948
- R? (x2): footprint Resistor_SMD:R_0402_1005Metric -> Resistor_SMD:R_0603_1608Metric
- R?: MPN C17514 -> (none)
- R? (x6): MPN C104384 -> (none)
- U1: LCSC (none) -> C5250982
- U4: LCSC (none) -> C85364
- Y1: footprint Crystal:Crystal_SMD_HC49-SD -> Crystal:Crystal_SMD_3225-4Pin_3.2x2.5mm; LCSC (none) -> C9002
Connections:
- net GND: now also Y1.2, Y1.4
- net USB_DN: now reaches R?.2, U?.46 (USB_DM)
- net USB_DP: now reaches R?.2, U?.47 (USB_DP)
Other:
- moved on the sheet: R?
Changed lines of the file:
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@@
   (junction (at 245.11 129.54) (diameter 0) (color 0 0 0 0)
   )
+  (junction (at 38.1 193.04) (diameter 0) (color 0 0 0 0)
+  )
   (junction (at 118.11 257.81) (diameter 0) (color 0 0 0 0)
   )
@@
     (stroke (width 0) (type default))
   )
+  (wire (pts (xy 43.18 193.04) (xy 38.1 193.04))
+    (stroke (width 0) (type default))
+  )
   (wire (pts (xy 279.4 124.46) (xy 288.29 124.46))
     (stroke (width 0) (type default))
@@
     (stroke (width 0) (type default))
   )
-  (wire (pts (xy 308.61 152.4) (xy 322.58 152.4))
+  (wire (pts (xy 317.5 154.94) (xy 331.47 154.94))
     (stroke (width 0) (type default))
   )
@@
     (stroke (width 0) (type default))
   )
-  (wire (pts (xy 294.64 152.4) (xy 300.99 152.4))
-    (stroke (width 0) (type default))
-  )
   (bus (pts (xy 334.01 187.96) (xy 334.01 190.5))
     (stroke (width 0) (type default))
@@
     (stroke (width 0) (type default))
   )
-  (wire (pts (xy 308.61 144.78) (xy 322.58 144.78))
+  (wire (pts (xy 317.5 147.32) (xy 331.47 147.32))
     (stroke (width 0) (type default))
   )
@@
     (stroke (width 0) (type default))
   )
+  (wire (pts (xy 33.02 184.15) (xy 33.02 193.04))
+    (stroke (width 0) (type default))
+  )
   (wire (pts (xy 49.53 125.73) (xy 58.42 125.73))
     (stroke (width 0) (type default))
@@
     (stroke (width 0) (type default))
   )
+  (wire (pts (xy 33.02 193.04) (xy 38.1 193.04))
+    (stroke (width 0) (type default))
+  )
   (wire (pts (xy 231.14 200.66) (xy 217.17 200.66))
     (stroke (width 0) (type default))
@@
     (stroke (width 0) (type default))
   )
+  (wire (pts (xy 309.88 152.4) (xy 294.64 152.4))
+    (stroke (width 0) (type default))
+  )
   (bus (pts (xy 334.01 167.64) (xy 334.01 170.18))
     (stroke (width 0) (type default))
@@
     (stroke (width 0) (type default))
   )
+  (wire (pts (xy 43.18 184.15) (xy 43.18 193.04))
+    (stroke (width 0) (type default))
+  )
   (bus (pts (xy 334.01 170.18) (xy 334.01 172.72))
     (stroke (width 0) (type default))
@@
     (stroke (width 0) (type default))
   )
-  (wire (pts (xy 294.64 149.86) (xy 300.99 149.86))
+  (wire (pts (xy 294.64 149.86) (xy 309.88 149.86))
     (stroke (width 0) (type default))
   )
@@
     (stroke (width 0) (type default))
   )
+  (wire (pts (xy 309.88 154.94) (xy 309.88 152.4))
+    (stroke (width 0) (type default))
+  )
+  (wire (pts (xy 38.1 193.04) (xy 38.1 194.31))
+    (stroke (width 0) (type default))
+  )
   (wire (pts (xy 73.66 106.68) (xy 68.58 106.68))
     (stroke (width 0) (type default))
@@
     (stroke (width 0) (type default))
   )
-  (wire (pts (xy 300.99 144.78) (xy 300.99 149.86))
+  (wire (pts (xy 309.88 147.32) (xy 309.88 149.86))
     (stroke (width 0) (type default))
   )
@@
     (effects (font (size 2.54 2.54)) (justify left bottom))
   )
-  (text "Make sure R4 and R6\nare close to RP2040" (at 308.61 149.86 0)
+  (text "Make sure R4 and R6\nare close to RP2040" (at 317.5 152.4 0)
     (effects (font (size 1.27 1.27)) (justify left bottom))
   )
@@
     (effects (font (size 1.27 1.27)) (justify right bottom))
   )
-  (label "USB_D+" (at 322.58 144.78 180) (fields_autoplaced)
+  (label "USB_D+" (at 331.47 147.32 180) (fields_autoplaced)
     (effects (font (size 1.27 1.27)) (justify right bottom))
   )
@@
     (effects (font (size 1.27 1.27)) (justify left bottom))
   )
+  (label "USB_DN" (at 309.88 152.4 180) (fields_autoplaced)
+    (effects (font (size 1.27 1.27)) (justify right bottom))
+  )
   (label "QSPI_SCLK" (at 125.73 262.89 0) (fields_autoplaced)
     (effects (font (size 1.27 1.27)) (justify left bottom))
@@
     (effects (font (size 1.27 1.27)) (justify right bottom))
   )
+  (label "USB_DP" (at 309.88 149.86 180) (fields_autoplaced)
+    (effects (font (size 1.27 1.27)) (justify right bottom))
+  )
   (label "XOUT" (at 76.2 189.23 180) (fields_autoplaced)
     (effects (font (size 1.27 1.27)) (justify right bottom))
@@
     (effects (font (size 1.27 1.27)) (justify right bottom))
   )
-  (label "USB_D-" (at 322.58 152.4 180) (fields_autoplaced)
+  (label "USB_D-" (at 331.47 154.94 180) (fields_autoplaced)
     (effects (font (size 1.27 1.27)) (justify right bottom))
   )
@@
     )
   )
-  (symbol (lib_id "arisu-rescue:R-Device") (at 304.8 144.78 270) (unit 1)
+  (symbol (lib_id "arisu-rescue:R-Device") (at 313.69 147.32 270) (unit 1)
     (in_bom yes) (on_board yes) (dnp no)
-    (property "Reference" "R?" (at 304.8 139.5222 90)
+    (property "Reference" "R?" (at 313.69 142.0622 90)
       (effects (font (size 1.27 1.27)))
     )
-    (property "Value" "27" (at 304.8 141.8336 90)
+    (property "Value" "27" (at 313.69 144.3736 90)
       (effects (font (size 1.27 1.27)))
     )
-    (property "Footprint" "Resistor_SMD:R_0402_1005Metric" (at 304.8 143.002 90)
+    (property "Footprint" "Resistor_SMD:R_0603_1608Metric" (at 313.69 145.542 90)
       (effects (font (size 1.27 1.27)) hide)
     )
-    (property "Datasheet" "~" (at 304.8 144.78 0)
+    (property "Datasheet" "~" (at 313.69 147.32 0)
       (effects (font (size 1.27 1.27)) hide)
     )
@@
     )
   )
-  (symbol (lib_id "arisu-rescue:R-Device") (at 304.8 152.4 270) (unit 1)
+  (symbol (lib_id "arisu-rescue:R-Device") (at 313.69 154.94 270) (unit 1)
     (in_bom yes) (on_board yes) (dnp no)
-    (property "Reference" "R?" (at 304.8 147.1422 90)
+    (property "Reference" "R?" (at 313.69 149.6822 90)
       (effects (font (size 1.27 1.27)))
     )
-    (property "Value" "27" (at 304.8 149.4536 90)
+    (property "Value" "27" (at 313.69 151.9936 90)
       (effects (font (size 1.27 1.27)))
     )
-    (property "Footprint" "Resistor_SMD:R_0402_1005Metric" (at 304.8 150.622 90)
+    (property "Footprint" "Resistor_SMD:R_0603_1608Metric" (at 313.69 153.162 90)
       (effects (font (size 1.27 1.27)) hide)
     )
-    (property "Datasheet" "~" (at 304.8 152.4 0)
+    (property "Datasheet" "~" (at 313.69 154.94 0)
       (effects (font (size 1.27 1.27)) hide)
     )
@@
       (effects (font (size 1.27 1.27)) hide)
     )
-    (property "MPN" "C17514" (at 30.48 148.59 0)
-      (effects (font (size 1.27 1.27)) hide)
-    )
     (pin "1")
     (pin "2")
@@
       (effects (font (size 1.27 1.27)))
     )
-    (property "Footprint" "Crystal:Crystal_SMD_HC49-SD" (at 38.1 184.15 0)
+    (property "Footprint" "Crystal:Crystal_SMD_3225-4Pin_3.2x2.5mm" (at 38.1 184.15 0)
       (effects (font (size 1.27 1.27)) hide)
     )
@@
       (effects (font (size 1.27 1.27)) hide)
     )
+    (property "LCSC" "C9002" (at 50.8 182.2197 0)
+      (effects (font (size 1.27 1.27)) hide)
+    )
     (pin "1")
     (pin "2")
@@
       (effects (font (size 1.27 1.27)) hide)
     )
-    (property "MPN" "C104384" (at 212.09 207.01 0)
-      (effects (font (size 1.27 1.27)) hide)
-    )
     (pin "1")
     (pin "2")
@@
       (effects (font (size 1.27 1.27)) hide)
     )
-    (property "MPN" "C104384" (at 118.11 250.19 0)
-      (effects (font (size 1.27 1.27)) hide)
-    )
     (pin "1")
     (pin "2")
@@
       (effects (font (size 1.27 1.27)) hide)
     )
+    (property "LCSC" "C20803" (at 66.04 102.87 0)
+      (effects (font (size 1.27 1.27)) hide)
+    )
     (pin "1")
     (pin "2")
@@
       (effects (font (size 1.27 1.27)) hide)
     )
+    (property "LCSC" "C165948" (at 34.29 100.33 0)
+      (effects (font (size 1.27 1.27)) hide)
+    )
     (pin "A1")
     (pin "A12")
@@
       (effects (font (size 1.27 1.27)) hide)
     )
-    (property "MPN" "C104384" (at 53.34 110.49 0)
-      (effects (font (size 1.27 1.27)) hide)
-    )
     (pin "1")
     (pin "2")
@@
       (effects (font (size 1.27 1.27)) hide)
     )
-    (property "MPN" "C104384" (at 118.11 238.76 0)
-      (effects (font (size 1.27 1.27)) hide)
-    )
     (pin "1")
     (pin "2")
@@
       (effects (font (size 1.27 1.27)) hide)
     )
+    (property "LCSC" "C5250982" (at 39.37 72.39 0)
+      (effects (font (size 1.27 1.27)) hide)
+    )
     (pin "1")
     (pin "2")
@@
       (effects (font (size 1.27 1.27)) hide)
     )
-    (property "MPN" "C104384" (at 53.34 115.57 0)
-      (effects (font (size 1.27 1.27)) hide)
-    )
     (pin "1")
     (pin "2")
@@
       (effects (font (size 1.27 1.27)) hide)
     )
+    (property "LCSC" "C85364" (at 123.7997 110.49 0)
+      (effects (font (size 1.27 1.27)) hide)
+    )
     (pin "1")
     (pin "2")
@@
     )
   )
+  (symbol (lib_id "arisu-rescue:GND-power") (at 38.1 194.31 0) (unit 1)
+    (in_bom yes) (on_board yes) (dnp no)
+    (property "Reference" "#PWR?" (at 38.1 200.66 0)
+      (effects (font (size 1.27 1.27)) hide)
+    )
+    (property "Value" "GND" (at 38.227 198.7042 0)
+      (effects (font (size 1.27 1.27)))
+    )
+    (property "Footprint" "" (at 38.1 194.31 0)
+      (effects (font (size 1.27 1.27)) hide)
+    )
+    (property "Datasheet" "" (at 38.1 194.31 0)
+      (effects (font (size 1.27 1.27)) hide)
+    )
+    (pin "1")
+    (instances
+      (project "RP2040_minimal"
+        (path "/4e80874f-13b9-4886-a592-f501191b7905"
+          (reference "#PWR?") (unit 1)
+        )
+      )
+      (project "arisu"
+        (path "/6a4507f9-fb93-401b-b9e1-9f2bcbbd5186"
+          (reference "#PWR034") (unit 1)
+        )
+      )
+    )
+  )
   (symbol (lib_id "arisu-rescue:R-Device") (at 212.09 195.58 0) (unit 1)
     (in_bom yes) (on_board yes) (dnp no)
@@
       (effects (font (size 1.27 1.27)) hide)
     )
-    (property "MPN" "C104384" (at 212.09 195.58 0)
-      (effects (font (size 1.27 1.27)) hide)
-    )

Commit message: Final Prototype 1
Connections:
- net +3V3: now also P1.1 (VTref)
- net +5V: no longer P1.1 (VTref)
- net GND: no longer P1.5 (GND)
- no-connect marks 6 -> 8
Changed lines of the file:
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@@
   (no_connect (at 49.53 134.62))
   (no_connect (at 133.35 127))
+  (no_connect (at 34.29 271.78))
   (no_connect (at 44.45 259.08))
+  (no_connect (at 44.45 264.16))
   (bus_entry (at 331.47 228.6) (size 2.54 2.54)
     (stroke (width 0) (type default))
@@
     (stroke (width 0) (type default))
   )
+  (wire (pts (xy 218.44 227.33) (xy 231.14 227.33))
+    (stroke (width 0) (type default))
+  )
   (wire (pts (xy 217.17 195.58) (xy 231.14 195.58))
     (stroke (width 0) (type default))
@@
     (stroke (width 0) (type default))
   )
-  (wire (pts (xy 218.44 228.6) (xy 218.44 227.33))
-    (stroke (width 0) (type default))
-  )
   (wire (pts (xy 311.15 118.11) (xy 311.15 120.65))
     (stroke (width 0) (type default))
@@
     (stroke (width 0) (type default))
   )
-  (wire (pts (xy 218.44 223.52) (xy 218.44 224.79))
-    (stroke (width 0) (type default))
-  )
   (wire (pts (xy 275.59 142.24) (xy 275.59 129.54))
     (stroke (width 0) (type default))
@@
     (stroke (width 0) (type default))
   )
-  (wire (pts (xy 218.44 227.33) (xy 231.14 227.33))
-    (stroke (width 0) (type default))
-  )
   (wire (pts (xy 279.4 109.22) (xy 279.4 124.46))
     (stroke (width 0) (type default))
@@
     (stroke (width 0) (type default))
   )
-  (wire (pts (xy 218.44 228.6) (xy 217.17 228.6))
-    (stroke (width 0) (type default))
-  )
   (wire (pts (xy 217.17 167.64) (xy 231.14 167.64))
     (stroke (width 0) (type default))
@@
     (stroke (width 0) (type default))
   )
-  (wire (pts (xy 218.44 223.52) (xy 217.17 223.52))
-    (stroke (width 0) (type default))
-  )
   (bus (pts (xy 334.01 200.66) (xy 334.01 203.2))
     (stroke (width 0) (type default))
@@
     (effects (font (size 1.27 1.27)) (justify right bottom))
   )
-  (label "SWDIO" (at 220.98 227.33 0) (fields_autoplaced)
+  (label "SWDIO" (at 218.44 227.33 0) (fields_autoplaced)
     (effects (font (size 1.27 1.27)) (justify left bottom))
   )
@@
     (effects (font (size 1.27 1.27)) (justify right bottom))
   )
-  (label "SWCLK" (at 220.98 224.79 0) (fields_autoplaced)
+  (label "SWCLK" (at 218.44 224.79 0) (fields_autoplaced)
     (effects (font (size 1.27 1.27)) (justify left bottom))
   )
@@
     (effects (font (size 1.27 1.27)) (justify right bottom))
   )
-  (global_label "SWCLK" (shape input) (at 217.17 223.52 180) (fields_autoplaced)
-    (effects (font (size 1.27 1.27)) (justify right))
-    (property "Intersheetrefs" "${INTERSHEET_REFS}" (at 208.6894 223.52 0)
-      (effects (font (size 1.27 1.27)) (justify right) hide)
-    )
-  )
-  (global_label "SWDIO" (shape input) (at 217.17 228.6 180) (fields_autoplaced)
-    (effects (font (size 1.27 1.27)) (justify right))
-    (property "Intersheetrefs" "${INTERSHEET_REFS}" (at 209.0522 228.6 0)
-      (effects (font (size 1.27 1.27)) (justify right) hide)
-    )
-  )
   (symbol (lib_id "arisu-rescue:SW_Push-Switch") (at 203.2 210.82 0) (unit 1)
     (in_bom yes) (on_board yes) (dnp no)
@@
     )
   )
+  (symbol (lib_id "PCM_RP2040_minimal-rescue:+3V3-power") (at 31.75 241.3 0) (unit 1)
+    (in_bom yes) (on_board yes) (dnp no)
+    (property "Reference" "#PWR?" (at 31.75 245.11 0)
+      (effects (font (size 1.27 1.27)) hide)
+    )
+    (property "Value" "+3V3" (at 32.131 236.9058 0)
+      (effects (font (size 1.27 1.27)))
+    )
+    (property "Footprint" "" (at 31.75 241.3 0)
+      (effects (font (size 1.27 1.27)) hide)
+    )
+    (property "Datasheet" "" (at 31.75 241.3 0)
+      (effects (font (size 1.27 1.27)) hide)
+    )
+    (pin "1")
+    (instances
+      (project "RP2040_minimal"
+        (path "/4e80874f-13b9-4886-a592-f501191b7905"
+          (reference "#PWR?") (unit 1)
+        )
+      )
+      (project "arisu"
+        (path "/6a4507f9-fb93-401b-b9e1-9f2bcbbd5186"
+          (reference "#PWR04") (unit 1)
+        )
+      )
+    )
+  )
   (symbol (lib_id "arisu-rescue:R-Device") (at 30.48 148.59 270) (unit 1)
     (in_bom yes) (on_board yes) (dnp no)
@@
         )
       )
-    )
-  )
-  (symbol (lib_id "power:+5V") (at 31.75 241.3 0) (unit 1)
-    (in_bom yes) (on_board yes) (dnp no) (fields_autoplaced)
-    (property "Reference" "#PWR04" (at 31.75 245.11 0)
-      (effects (font (size 1.27 1.27)) hide)
-    )
-    (property "Value" "+5V" (at 31.75 237.49 0)
-      (effects (font (size 1.27 1.27)))
-    )
-    (property "Footprint" "" (at 31.75 241.3 0)
-      (effects (font (size 1.27 1.27)) hide)
-    )
-    (property "Datasheet" "" (at 31.75 241.3 0)
-      (effects (font (size 1.27 1.27)) hide)
-    )
-    (pin "1")
-    (instances
-      (project "arisu"
-        (path "/6a4507f9-fb93-401b-b9e1-9f2bcbbd5186"
-          (reference "#PWR04") (unit 1)
-        )
-      )
