File: PCB files/blossom_pcb/LED_backlight_matrix.kicad_sch (KiCad schematic)
At the start: 9 parts

Commit message: Possible final
Parts:
- R101: LCSC (none) -> C270888
Changed lines of the file:
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@@
+      (effects (font (size 1.27 1.27)) hide)
+    )
+    (property "LCSC" "C270888" (at 119.38 25.2222 0)
       (effects (font (size 1.27 1.27)) hide)
     )
